File: IO_UI.kicad_sch (KiCad schematic)
At the start: 20 parts, among them J1 USB_A, J2 USB_A, J4 USB_B_Micro, J5 USB_C_Receptacle_USB2.0_16P, Q1 PMOS, Q2 NMOS, Q3 NMOS, Q4 PMOS

Commit message: gerber command
Parts:
- J5: footprint Connector_USB:USB_C_Receptacle_HRO_TYPE-C-31-M-12 -> Connector_USB:USB_C_Receptacle_HCTL_HC-TYPE-C-16P-01A
Changed lines of the file:
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@@
 			)
 		)
-		(property "Footprint" "Connector_USB:USB_C_Receptacle_HRO_TYPE-C-31-M-12"
+		(property "Footprint" "Connector_USB:USB_C_Receptacle_HCTL_HC-TYPE-C-16P-01A"
 			(at 71.12 43.18 0)
 			(effects
