File: POWER_SOC.kicad_sch (KiCad schematic)
At the start: 31 parts, among them J3 Conn_01x02_Pin, J6 Conn_01x02_Pin, SW1 SW_Push

Commit message: gerber command
Parts:
- removed J3, J6: Conn_01x02_Pin, NetTie:NetTie-2_SMD_Pad2.0mm, symbol Connector:Conn_01x02_Pin
Connections:
- no-connect marks 1 -> 0
