File: power_bank.kicad_pcb (KiCad board)
At the start: 4 copper layers, 54.6 x 25.5 mm, 53 parts, among them J1 USB_A, J2 USB_A, J4 USB_B_Micro, J5 USB_C_Receptacle_USB2.0_16P, Q1 PMOS, Q2 NMOS, Q3 NMOS, Q4 PMOS, SW1 SW_Push

Commit message: gerber command
Parts:
- J5: footprint Connector_USB:USB_C_Receptacle_HRO_TYPE-C-31-M-12 -> Connector_USB:USB_C_Receptacle_HCTL_HC-TYPE-C-16P-01A
- moved G*** 4.56 mm to (132.9, 97.2)
Routing:
- net GND: track 157.0 -> 73.0 mm, vias 44 -> 11
- net LED3: track 25.4 -> 23.4 mm
- net VBUS: track 54.9 -> 54.3 mm
- added copper zone on B.Cu, net GND
- added copper zone on F.Cu, net GND
- removed copper zone on B.Cu, net (none)
- removed copper zone on F.Cu, net (none)
